File: eagle/chaoswest-token.brd (EAGLE design)
At the start: 44 x 50.7 mm, 40 parts, among them J1 USB, J2 ISP, Q1 Si1967DH, SW1 SSAJ120100, U1 MCP73832T-2ACI/OT, U2 ATTINY85V-10SU, U3 MCP9700AT-E/LT

Commit message: put the bottom silk screen (component names) into place
Parts:
- renumbered B+ to +

Commit message: current (hopefully nearly final) state of the PCB, minor changes, gerber files produced
Routing:
- net GND: track 269.1 -> 269.9 mm
Other:
- board text added: "git.io/cwtkn"
