File: eagle/rev-b/chaoswest-token.brd (EAGLE design)
At the start: 44 x 50.7 mm, 40 parts, among them J1 USB, J2 ISP, Q1 Si1967DH, SW1 SSAJ120100, U1 MCP73832T-2ACI/OT, U2 ATTINY85V-10SU, U3 MCP9700AT-E/LT

Commit message: Rev B Hardware completed and ordered
Parts:
- SW1: value SSAJ120100 -> SLIDE_BUTTONAYZ0102AGRLC; device extra:SSAJ120100 -> extra:AYZ0102AGRLC
- moved SW1 0.25 mm to (42.4, 34.0)
Connections:
- net +5V: no longer R7.2
- net VCC: now also R7.2
Routing:
- net VCC: track 231.2 -> 235.6 mm
- net N$6: track 9.45 -> 11.8 mm
- net VBAT: track 33.3 -> 31.3 mm
- net +5V: track 20.5 -> 18.8 mm
