File: eagle/rev-b/chaoswest-token.sch (EAGLE design)
At the start: 40 parts, among them J1 USB, J2 ISP, Q1 Si1967DH, SW1 SSAJ120100, U1 MCP73832T-2ACI/OT, U2 ATTINY85V-10SU, U3 MCP9700AT-E/LT

Commit message: Rev B Hardware completed and ordered
Parts:
- SW1: value SSAJ120100 -> SLIDE_BUTTONAYZ0102AGRLC; device extra:SSAJ120100 -> extra:SLIDE_BUTTONAYZ0102AGRLC
Connections:
- net +5V: no longer R7.2
- net VCC: now also R7.2
